Commit message: 1125

File: mando_description/urdf/scout_mini/scout_mini_carto.xacro (robot description, xacro)
@@ -1,5 +1,5 @@
 <?xml version='1.0'?>
-<robot name="atom_target" xmlns:xacro="http://www.ros.org/wiki/xacro">
-	<xacro:property name="robot_name" value="atom_target" />
+<robot name="atom" xmlns:xacro="http://www.ros.org/wiki/xacro">
+	<xacro:property name="robot_name" value="atom" />
 	<!-- <xacro:property name="robot_chassis_mass" value="15"/> -->
 	<xacro:property name="robot_chassis_mass" value="15" />
@@ -35,6 +35,7 @@
 	<xacro:property name="camera_mass" value="0.1" />
 	<xacro:property name="hokoyu_mass" value="1e-5" />
+	<xacro:arg name="frame" default="" />
 	<!-- Project center to the ground -->
-	<link name="base_footprint_target">
+	<link name="base_footprint">
 		<visual>
 			<origin xyz="0 0 0.0" rpy="1.57 0 -1.57" />
@@ -47,9 +48,10 @@
 			<geometry>
 				<mesh filename="package://mando_description/meshes/scout_mini/scout_mini_base_link2.dae" />
+				<!-- <box size="0.5 0.5 0.2"/> -->
 			</geometry>
 		</collision>
 	</link>
 	<!-- Make Chassis of Bot (Inertia Link) -->
-	<link name="chassis_target">
+	<link name="chassis">
 		<inertial>
 			<mass value="50" />
@@ -66,9 +68,16 @@
 		</inertial>
 	</link>
-	<!-- Robot base + Inertia  -->
+	<link name="base_link">
+	</link>
 	<joint name="base_footprint_joint" type="fixed">
 		<origin xyz="0 0 0" rpy="0 0 0" />
-		<parent link="base_footprint_target" />
-		<child link="chassis_target" />
+		<parent link="base_footprint" />
+		<child link="base_link" />
+	</joint>
+	<!-- Robot base + Inertia  -->
+	<joint name="base_link_joint" type="fixed">
+		<origin xyz="0 0 0" rpy="0 0 0" />
+		<parent link="base_link" />
+		<child link="chassis" />
 	</joint>
 	<!-- ixx="0.7171" ixy="0.0" ixz="0.0"
@@ -76,5 +85,5 @@
 				izz="0.1361" -->
 	<!-- Right Wheel Back -->
-	<link name="right_wheel_back_target">
+	<link name="right_wheel_back">
 		<inertial>
 			<mass value="${robot_wheel_mass}" />
@@ -99,5 +108,5 @@
 	</link>
 	<!-- Right Wheel Front-->
-	<link name="right_wheel_front_target">
+	<link name="right_wheel_front">
 		<inertial>
 			<mass value="${robot_wheel_mass}" />
@@ -122,5 +131,5 @@
 	</link>
 	<!-- Left wheel Back-->
-	<link name="left_wheel_back_target">
+	<link name="left_wheel_back">
 		<inertial>
 			<mass value="${robot_wheel_mass}" />
@@ -145,5 +154,5 @@
 	</link>
 	<!-- Left wheel Front-->
-	<link name="left_wheel_front_target">
+	<link name="left_wheel_front">
 		<inertial>
 			<mass value="${robot_wheel_mass}" />
@@ -168,5 +177,5 @@
 	</link>
 	<!-- Camera -->
-	<link name="camera_target">
+	<link name="camera">
 		<inertial>
 			<mass value="${camera_mass}" />
@@ -212,5 +221,5 @@
 	</link> -->
 	<!-- 2D Lidar  -->
-	<link name="base_scan_target">
+	<link name="base_scan">
 		<visual>
 			<origin xyz="0 0 0.0" rpy="0 0 0" />
@@ -233,18 +242,18 @@
 	</link>
 	<joint name="scan_joint" type="fixed">
-		<parent link="chassis_target" />
-		<child link="base_scan_target" />
+		<parent link="chassis" />
+		<child link="base_scan" />
 		<origin xyz="-0.032 0 0.172" rpy="0 0 0" />
 	</joint>
 	<!-- IMU Sensor -->
 	<joint name="imu_joint" type="fixed">
-		<parent link="chassis_target" />
-		<child link="imu_link_target" />
+		<parent link="chassis" />
+		<child link="imu_link" />
 		<origin xyz="0 0 0" rpy="0 0 0" />
 	</joint>
-	<link name="imu_link_target" />
+	<link name="imu_link" />
 	<!-- 3D Lidar Velodyne  -->
 	<xacro:include filename="$(find velodyne_description)/urdf/VLP-16.urdf.xacro" />
-	<xacro:VLP-16 parent="chassis_target" name="velodyne_target" topic="/velodyne_points_target" hz="10" samples="440">
+	<xacro:VLP-16 parent="chassis" name="velodyne" topic="/velodyne_points" hz="10" samples="440">
 		<origin xyz="0 0 0.4" rpy="0 0 0" />
 	</xacro:VLP-16>
@@ -254,6 +263,6 @@
 		<!-- <origin xyz="-0.2 -0.30 0" rpy="0 0 0" /> -->
 		<origin xyz="${-wheelbase/2} ${-track/2} ${wheel_vertical_offset}" rpy="0 0 0" />
-		<parent link="chassis_target" />
-		<child link="right_wheel_back_target" />
+		<parent link="chassis" />
+		<child link="right_wheel_back" />
 		<axis xyz="0 1 0" rpy="0 0 0" />
 		<!-- <limit effort="10000" velocity="1000" />
@@ -264,6 +273,6 @@
 		<!-- <origin xyz="0.2 -0.30 0" rpy="0 0 0" /> -->
 		<origin xyz="${wheelbase/2} ${-track/2} ${wheel_vertical_offset}" rpy="0 0 0" />
-		<parent link="chassis_target" />
-		<child link="right_wheel_front_target" />
+		<parent link="chassis" />
+		<child link="right_wheel_front" />
 		<axis xyz="0 1 0" rpy="0 0 0" />
 		<!-- <limit effort="10000" velocity="1000" />
@@ -274,6 +283,6 @@
 		<!-- <origin xyz="-0.2 0.30 0" rpy="0 0 0" /> -->
 		<origin xyz="${-wheelbase/2} ${track/2} ${wheel_vertical_offset}" rpy="0 0 0" />
-		<parent link="chassis_target" />
-		<child link="left_wheel_back_target" />
+		<parent link="chassis" />
+		<child link="left_wheel_back" />
 		<axis xyz="0 1 0" rpy="0 0 0" />
 		<!-- <limit effort="10000" velocity="1000" />
@@ -284,6 +293,6 @@
 		<!-- <origin xyz="0.2 0.30 0" rpy="0 0 0" /> -->
 		<origin xyz="${wheelbase/2} ${track/2} ${wheel_vertical_offset}" rpy="0 0 0" />
-		<parent link="chassis_target" />
-		<child link="left_wheel_front_target" />
+		<parent link="chassis" />
+		<child link="left_wheel_front" />
 		<axis xyz="0 1 0" rpy="0 0 0" />
 		<!-- <limit effort="10000" velocity="1000" />
@@ -293,6 +302,6 @@
 	<joint name="camera_joint" type="fixed">
 		<origin xyz="0.26 0 0" rpy="0 0 0" />
-		<parent link="chassis_target" />
-		<child link="camera_target" />
+		<parent link="chassis" />
+		<child link="camera" />
 		<axis xyz="0 1 0" />
 	</joint>
@@ -304,12 +313,12 @@
 	    <axis xyz="0 1 0"/>
 	</joint> -->
-	<gazebo reference="camera_target">
+	<gazebo reference="camera">
 		<!-- <material>Gazebo/Red</material> -->
 	</gazebo>
-	<gazebo reference="chassis_target">
+	<gazebo reference="chassis">
 		<!-- <material>Gazebo/Blue</material> -->
 	</gazebo>
 	<!-- Color of bot -->
-	<gazebo reference="left_wheel_front_target">
+	<gazebo reference="left_wheel_front">
 		<!-- <material>Gazebo/Green</material> -->
 		<kp>100000000</kp> <!-- kp and kd for rubber -->
@@ -320,5 +329,5 @@
 		<minDepth>0.00</minDepth>
 	</gazebo>
-	<gazebo reference="left_wheel_back_target">
+	<gazebo reference="left_wheel_back">
 		<!-- <material>Gazebo/Green</material> -->
 		<kp>100000000</kp> <!-- kp and kd for rubber -->
@@ -329,5 +338,5 @@
 		<minDepth>0.00</minDepth>
 	</gazebo>
-	<gazebo reference="right_wheel_front_target">
+	<gazebo reference="right_wheel_front">
 		<!-- <material>Gazebo/Green</material> -->
 		<kp>100000000</kp> <!-- kp and kd for rubber -->
@@ -338,5 +347,5 @@
 		<minDepth>0.00</minDepth>
 	</gazebo>
-	<gazebo reference="right_wheel_back_target">
+	<gazebo reference="right_wheel_back">
 		<!-- <material>Gazebo/Green</material> -->
 		<kp>100000000</kp> <!-- kp and kd for rubber -->
@@ -348,4 +357,4 @@
 	</gazebo>
 	<!-- Motor, Camera and Lidar Simulation -->
-	<xacro:include filename="$(find mando_description)/urdf/scout_mini/scout_mini_target.gazebo" />
+	<xacro:include filename="$(find mando_description)/urdf/scout_mini/scout_mini_carto.gazebo" />
 </robot>
